File: KiCad/Drone/Drone.kicad_pcb (KiCad board)
At the start: 2 copper layers, 91.4 x 57.1 mm, 22 parts, among them J1 ESC, J10 to ESC Power, J11 Conn_01x02_Female, J2 BATTRY, J3 ESP32_LEFT, J4 Raspberry Pi, J5 ESP32_RIGHT, J6 DPS310_LEFT, J7 US-015, J8 MPU9250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

Commit message: :+1:update schematic
Parts:
- added D3: SS2040FL, Diode_SMD:D_SOD-123F, B.Cu at (152.5, 87.6)
- added D4: SS2040FL, Diode_SMD:D_SOD-123F, B.Cu at (156.8, 87.0)
- added D5: SS2040FL, Diode_SMD:D_SOD-123F, B.Cu at (153.7, 108.0)
- added D6: SS2040FL, Diode_SMD:D_SOD-123F, B.Cu at (101.6, 118.7)
- added D7: UDZV5.1B, Diode_SMD:D_SOD-323, B.Cu at (151.1, 108.0)
- added R1: 1k, Resistor_SMD:R_0603_1608Metric_Pad1.05x0.95mm_HandSolder, B.Cu at (135.7, 86.4)
- added R2: 10k, Resistor_SMD:R_0603_1608Metric_Pad1.05x0.95mm_HandSolder, B.Cu at (159.8, 88.3)
- added R3: 10k, Resistor_SMD:R_0603_1608Metric_Pad1.05x0.95mm_HandSolder, F.Cu at (111.4, 94.6)
- added R4: 10k, Resistor_SMD:R_0603_1608Metric_Pad1.05x0.95mm_HandSolder, F.Cu at (113.7, 91.4)
- added R5: 10k, Resistor_SMD:R_0603_1608Metric_Pad1.05x0.95mm_HandSolder, F.Cu at (117.7, 99.1)
- added R6: 10k, Resistor_SMD:R_0603_1608Metric_Pad1.05x0.95mm_HandSolder, F.Cu at (120.3, 97.2)
- moved D1 1.81 mm to (160.0, 109.3), turned to 270 degrees
- moved C1 1.11 mm to (161.6, 105.9), turned to 270 degrees
- moved J2 0.67 mm to (172.7, 119.0)
Connections:
- C2 pad 1: 5V -> Net-(C2-Pad1)
- J3 pad 19: 5V -> Net-(D6-Pad1)
- L1 pad 2: 5V -> Net-(C2-Pad1)
- U1 pad 4: 5V -> Net-(C2-Pad1)
- U2 pad 1: GPIO21 -> Net-(D3-Pad2)
Routing:
- net Net-(D3-Pad2): track 0.00 -> 38.3 mm
- net GPIO21: track 33.8 -> 2.60 mm, vias 1 -> 0
- net GND: track 124.6 -> 146.9 mm
- net Net-(C2-Pad1): track 0.00 -> 17.7 mm
- net 5V: track 170.9 -> 183.6 mm, vias 0 -> 1
- net BAT: track 94.3 -> 84.1 mm
- net GPIO4: track 31.1 -> 35.2 mm
- net Net-(D6-Pad1): track 0.00 -> 3.05 mm
- net GPIO15: track 30.3 -> 28.4 mm
- net GPIO17: track 37.4 -> 38.3 mm
Other:
- board text added: "USB↓"

Commit message: :+1:update schematic ver3
Parts:
- removed the screw at (140.9, 105.7)
- removed the screw at (120.8, 105.7)
- added C4: 0.1uF, Capacitor_SMD:C_0603_1608Metric, F.Cu at (106.7, 126.5)
- added C5: 0.1uF, Capacitor_SMD:C_0603_1608Metric, F.Cu at (101.4, 116.2)
- added C6: 22uF, Capacitor_SMD:C_0603_1608Metric, F.Cu at (101.4, 118.1)
- added C7: 0.1uF, Capacitor_SMD:C_0603_1608Metric, F.Cu at (106.8, 114.3)
- added R7: 10k, Resistor_SMD:R_0603_1608Metric_Pad1.05x0.95mm_HandSolder, F.Cu at (117.2, 92.1)
- added R8: 10k, Resistor_SMD:R_0603_1608Metric_Pad1.05x0.95mm_HandSolder, F.Cu at (101.4, 114.3)
- added SW1: SW_Push, Button_Switch_THT:SW_PUSH_6mm, F.Cu at (112.4, 85.1)
- added U3: ESP32-WROOM-32, RF_Module:ESP32-WROOM-32, F.Cu at (108.0, 102.9)
- added screw: MountingHole_3mm, MountingHole:MountingHole_3mm, F.Cu at (143.4, 108.2)
- added screw: MountingHole_3mm, MountingHole:MountingHole_3mm, F.Cu at (123.3, 108.3)
- D6, R1: moved to F.Cu
- J3: value ESP32_LEFT -> AZ1086H-3.3; footprint Connector_PinSocket_2.54mm:PinSocket_1x19_P2.54mm_Vertical -> Package_TO_SOT_SMD:SOT-223-3_TabPin2; moved to F.Cu
- J5: value ESP32_RIGHT -> Conn_01x06_Female; footprint Connector_PinSocket_2.54mm:PinSocket_1x19_P2.54mm_Vertical -> Connector_PinHeader_2.54mm:PinHeader_1x06_P2.54mm_Horizontal; moved to F.Cu
- R3, R4, R5, R6: moved to B.Cu
- moved J3 41.5 mm to (106.7, 122.6), turned to 0 degrees
- moved C3 41.3 mm to (104.1, 115.1), turned to 90 degrees
- moved J5 40.3 mm to (128.3, 124.5), turned to 270 degrees
- moved J9 32.4 mm to (132.1, 83.8), turned to 0 degrees
- moved R1 30.0 mm to (106.0, 91.0), turned to 270 degrees
- moved D6 21.7 mm to (123.2, 120.7)
- moved J6 18.1 mm to (121.9, 83.8), turned to 0 degrees
- moved R4 16.9 mm to (101.0, 102.6), turned to 90 degrees
- moved R6 16.2 mm to (106.0, 105.0), turned to 90 degrees
- moved R5 15.0 mm to (103.5, 103.9), turned to 90 degrees
- moved R3 14.8 mm to (98.4, 101.8), turned to 90 degrees
- moved J7 11.1 mm to (127.0, 116.2), turned to 90 degrees
- moved R2 10.0 mm to (168.3, 93.6), turned to 270 degrees
- moved C2 8.13 mm to (152.4, 101.6), turned to 180 degrees
- moved J11 6.25 mm to (142.2, 116.2)
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Connections:
- C3 pad 2: EN -> ESP_EN
- D6 pad 1: Net-(D6-Pad1) -> 5V
- D6 pad 2: 5V -> Net-(D6-Pad2)
- J1 pad 3: GPIO15 -> GPIO17
- J1 pad 4: GPIO4 -> GPIO16
- J1 pad 5: GPIO16 -> GPIO4
- J1 pad 6: GPIO17 -> GPIO15
- J3 pad 1: 3V3 -> GND
- J3 pad 2: EN -> 3V3
- J3 pad 3: VP -> 5V
- J4 pad 7: PI_UART_TX -> ESP_TX
- J4 pad 9: PI_UART_RX -> ESP_RX
- J5 pad 2: GPIO23 -> Net-(J5-Pad2)
- J5 pad 3: GPIO22 -> Net-(D6-Pad2)
- J5 pad 4: PI_UART_RX -> ESP_TX
- J5 pad 5: PI_UART_TX -> ESP_RX
- J5 pad 6: GPIO21 -> Net-(C7-Pad2)
- R3 pad 1: GPIO15 -> GPIO17
- R4 pad 1: GPIO4 -> GPIO16
- R5 pad 1: GPIO16 -> GPIO4
- R6 pad 1: GPIO17 -> GPIO15
Routing:
- net ESP_TX: track 0.00 -> 59.5 mm, vias 0 -> 1
- net ESP_RX: track 0.00 -> 57.7 mm, vias 0 -> 1
- net Net-(D3-Pad2): track 38.3 -> 77.7 mm, vias 0 -> 1
- net PI_UART_TX: track 36.9 -> 0.00 mm
- net PI_UART_RX: track 36.2 -> 0.00 mm
- net 5V: track 183.6 -> 152.8 mm
- net GND: track 146.9 -> 123.8 mm, vias 16 -> 19
- net CSBN: track 17.3 -> 36.5 mm, vias 0 -> 1
- net GPIO17: track 38.3 -> 21.3 mm, vias 2 -> 1
- net Net-(R7-Pad2): track 0.00 -> 15.4 mm
- net Net-(C7-Pad2): track 0.00 -> 13.5 mm, vias 0 -> 1
- net GPIO5: track 6.13 -> 18.3 mm, vias 0 -> 1
- net Echo: track 6.35 -> 18.6 mm
- net GPIO4: track 35.2 -> 24.7 mm
- net GPIO16: track 33.1 -> 23.0 mm
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Other:
- board text added: "DRONE_PROJECT CIRCUIT_BOARD_V3"
- board text added: "RX"
- board text added: "TX"
- board text removed: "DRONE_PROJECT CIRCUIT_BOARD_V2"
- board text removed: "ESP32 DevkitC"
- board text removed: "USB↓"

Commit message: :+1:fixed footprint
Parts:
- moved C4 11.4 mm to (97.3, 120.0), turned to 180 degrees
Changed lines of the file:
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@@
   )
   (module Capacitor_SMD:C_0603_1608Metric (layer F.Cu)
-    (at 106.68 126.5175 270)
+    (at 97.3075 120.015 180)
     (descr "Capacitor SMD 0603 (1608 Metric), square (rectangular) end terminal, IPC_7351 nominal, (Body size source: http://www.tortai-tech.com/upload/download/2011102023233369053.pdf), generated with kicad-footprint-generator")
     (tags capacitor)
     (attr smd)
-    (fp_text reference C4 (at 0 -1.43 90) (layer F.SilkS)
+    (fp_text reference C4 (at 0 -1.43) (layer F.SilkS)
       (effects (font (size 1 1) (thickness 0.15)))
     )
-    (fp_text value 0.1uF (at 0 1.43 90) (layer F.Fab)
+    (fp_text value 0.1uF (at 0 1.43) (layer F.Fab)
       (effects (font (size 1 1) (thickness 0.15)))
     )
-    (fp_text user %R (at 0 0 90) (layer F.Fab)
+    (fp_text user %R (at 0 0) (layer F.Fab)
       (effects (font (size 0.4 0.4) (thickness 0.06)))
     )
@@
     (fp_line (start -0.8 -0.4) (end 0.8 -0.4) (layer F.Fab) (width 0.1))
     (fp_line (start -0.8 0.4) (end -0.8 -0.4) (layer F.Fab) (width 0.1))
-    (pad 2 smd roundrect (at 0.7875 0 270) (size 1 1.1) (layers F.Cu F.Paste F.Mask) (roundrect_rratio 0.25)
+    (pad 2 smd roundrect (at 0.7875 0 180) (size 1 1.1) (layers F.Cu F.Paste F.Mask) (roundrect_rratio 0.25)
       (net 1 GND))
-    (pad 1 smd roundrect (at -0.7875 0 270) (size 1 1.1) (layers F.Cu F.Paste F.Mask) (roundrect_rratio 0.25)
+    (pad 1 smd roundrect (at -0.7875 0 180) (size 1 1.1) (layers F.Cu F.Paste F.Mask) (roundrect_rratio 0.25)
       (net 3 5V))
     (model ${KISYS3DMOD}/Capacitor_SMD.3dshapes/C_0603_1608Metric.wrl
